File: capstone_pcb.kicad_sch (KiCad schematic)
At the start: 47 parts, among them IC6 BSS138, Q1 BSS138, U2 BMI270, U3 NRF52840-QIAA-R, U4 MAX30102EFD+T, U5 AMS1117-1.8, U6 TPS61099DRV, X1 32MHz, X2 32.768kHz

Commit message: add LCSC part numbers
Parts:
- BT1: LCSC (none) -> C70379
- C1, C17, C18: LCSC (none) -> C1547
- C11: LCSC (none) -> C1546
- C12, C16, C21, C5, C7, C8: LCSC (none) -> C1525
- C14: LCSC (none) -> C52923
- C15: footprint Capacitor_SMD:C_0201_0603Metric -> Capacitor_SMD:C_0402_1005Metric; LCSC (none) -> C529923
- C19, C20, C6: LCSC (none) -> C23733
- C2: footprint Capacitor_SMD:C_0201_0603Metric -> Capacitor_SMD:C_0402_1005Metric; LCSC (none) -> C1547
- C23: value 0.1uF -> 100nF; LCSC (none) -> C1525
- C24, C25, C26: LCSC (none) -> C15525
- C3: LCSC (none) -> C40459
- C4: LCSC (none) -> C1544
- C9: LCSC (none) -> C1543
- IC6, Q1: LCSC (none) -> C52895
- L1: footprint Inductor_SMD:L_0201_0603Metric -> Inductor_SMD:L_0402_1005Metric; LCSC (none) -> C13595
- L2: footprint (none) -> Inductor_SMD:L_0402_1005Metric; LCSC (none) -> C49067
- R1, R2: LCSC (none) -> C25900
- R3, R4, R5, R6, R7: LCSC (none) -> C25531
- R8: value 1.35M -> 453k; LCSC (none) -> C27009
- R9: value 300k -> 100k; LCSC (none) -> C25530
- U2: LCSC (none) -> C2836813
- U3: LCSC (none) -> C190794
- U4: LCSC (none) -> C6454833
- U5: LCSC (none) -> C347220
- U6: LCSC (none) -> C2842395
- X1: footprint Crystal:Crystal_SMD_3215-2Pin_3.2x1.5mm -> Crystal:Crystal_SMD_3225-4Pin_3.2x2.5mm; LCSC (none) -> C1122385
- X2: LCSC (none) -> C32346
