File: capstone_pcb.kicad_sch (KiCad schematic)
At the start: 47 parts, among them IC6 BSS138, Q1 BSS138, U2 BMI270, U3 NRF52840-QIAA-R, U4 MAX30102EFD+T, U5 AMS1117-1.8, U6 TPS61099DRV, X1 32MHz, X2 32.768kHz

Commit message: exposed SWD pins and added LED for flashing status
Parts:
- added D1: LED, LED_SMD:LED_0402_1005Metric, symbol Device:LED
- added J2: Conn_01x05_Pin, Connector_PinHeader_1.27mm:PinHeader_2x05_P1.27mm_Vertical_SMD, symbol Connector:Conn_01x05_Pin
- added R10: 0.4k, Resistor_SMD:R_0402_1005Metric, symbol Device:R_US
- BT1: LCSC C70379 -> C5470546
- C15: LCSC C529923 -> C52923
- R3, R4, R5, R6, R7: value 10K -> 10k
- U3: footprint nrf:nrf52840_qiaa_r -> nrf:XCVR_NRF52840-QIAA-R-edited
Connections:
- net +3V3: now also J2.5 (Pin_5), R10.1
- net GND: now also J2.3 (Pin_3)
- net P0.13: no longer names the net of U3.AD8 (P0.13)
- net P0.13: now also D1.1 (K)
- net P0.18/RESET: no longer names the net of U3.AC13 (P0.18/NRESET)
- net P0.18/RESET: now also J2.1 (Pin_1)
- net SWDCLK: no longer names the net of U3.AA24 (SWDCLK)
- net SWDCLK: now also J2.4 (Pin_4)
- net SWDIO: no longer names the net of U3.AC24 (SWDIO)
- net SWDIO: now also J2.2 (Pin_2)
- new net: D1.2 (A), R10.2
- no-connect marks 60 -> 54
Other:
- moved on the sheet: C7, C9

Commit message: add silkscreen labels to pin header
Parts:
- removed J2: Conn_01x05_Pin, Connector_PinHeader_1.27mm:PinHeader_2x05_P1.27mm_Vertical_SMD, symbol Connector:Conn_01x05_Pin
- added J1: Conn_01x05, Connector_PinHeader_2.54mm:PinHeader_1x05_P2.54mm_Vertical, symbol Connector_Generic:Conn_01x05
Connections:
- net +3V3: now also J1.1 (Pin_1)
- net GND: now also J1.3 (Pin_3)
- net at U3.AC13 (P0.18/NRESET): now also J1.5 (Pin_5)
- net at U3.AC24 (SWDIO): now also J1.4 (Pin_4)
- net at U3.AA24 (SWDCLK): now also J1.2 (Pin_2)

Commit message: added 100k and 130k resistors in series
Parts:
- removed U6: TPS61099DRV, Package_SON:WSON-6-1EP_2x2mm_P0.65mm_EP1x1.6mm, symbol Regulator_Switching:TPS61099DRV
- added R11: 130k, Resistor_SMD:R_0402_1005Metric, symbol Device:R_US
- added U1: TPS610994DRV, Package_SON:WSON-6-1EP_2x2mm_P0.65mm_EP1x1.6mm, symbol Regulator_Switching:TPS610994DRV
- R8: value 453k -> 100k; LCSC C27009 -> C25530
Connections:
- net +3V: now also U1.4 (EN), U1.6 (VI)
- net +3V3: now also R11.1, U1.2 (VOUT); no longer R8.2
- net GND: now also U1.1 (GND), U1.7 (GND)
- net at R8.1: now also R11.2; no longer R9.1
- net at L2.2: now also U1.5 (SW)
- new net: R8.2, R9.1, U1.3 (FB)
Other:
- moved on the sheet: C25, C26

Commit message: rearrange cap. and resist. to correct locations
Connections:
- net +3V3: no longer U3.AD2 (VBUS)
- new net AD2: U3.AD2 (VBUS)
- no-connect marks 54 -> 57
Changed lines of the file:
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@@
   (no_connect (at 271.78 91.44))
   (no_connect (at 271.78 99.06))
+  (no_connect (at 176.53 167.64))
   (no_connect (at 271.78 114.3))
   (no_connect (at 271.78 93.98))
@@
   (no_connect (at 176.53 104.14))
   (no_connect (at 176.53 124.46))
+  (no_connect (at 176.53 165.1))
   (no_connect (at 271.78 101.6))
   (no_connect (at 123.19 232.41))
@@
   (no_connect (at 271.78 86.36))
   (no_connect (at 271.78 170.18))
+  (no_connect (at 176.53 170.18))
   (no_connect (at 176.53 129.54))
   (no_connect (at 48.26 55.88))
@@
     (stroke (width 0) (type default))
   )
-  (wire (pts (xy 120.65 134.62) (xy 102.87 134.62))
+  (wire (pts (xy 120.65 134.62) (xy 116.84 134.62))
     (stroke (width 0) (type default))
   )
@@
     (stroke (width 0) (type default))
   )
-  (wire (pts (xy 120.65 130.81) (xy 120.65 134.62))
-    (stroke (width 0) (type default))
-  )
   (wire (pts (xy 176.53 81.28) (xy 187.96 81.28))
     (stroke (width 0) (type default))
@@
   (label "OSCB" (at 90.17 76.2 180) (fields_autoplaced)
     (effects (font (size 1.27 1.27)) (justify right bottom))
+  )
+  (label "AD2" (at 176.53 165.1 0) (fields_autoplaced)
+    (effects (font (size 1.27 1.27)) (justify left bottom))
   )
   (label "INT1" (at 48.26 58.42 0) (fields_autoplaced)
@@
     )
   )
-  (global_label "+3V3" (shape input) (at 120.65 130.81 90) (fields_autoplaced)
-    (effects (font (size 1.27 1.27)) (justify left))
-    (property "Intersheetrefs" "${INTERSHEET_REFS}" (at 120.65 122.7448 90)
-      (effects (font (size 1.27 1.27)) (justify left) hide)
-    )
-  )
-  (global_label "+3V3" (shape input) (at 176.53 165.1 180) (fields_autoplaced)
-    (effects (font (size 1.27 1.27)) (justify right))
-    (property "Intersheetrefs" "${INTERSHEET_REFS}" (at 168.4648 165.1 0)
-      (effects (font (size 1.27 1.27)) (justify right) hide)
-    )
-  )
   (global_label "+1V8" (shape input) (at 66.04 218.44 90) (fields_autoplaced)
     (effects (font (size 1.27 1.27)) (justify left))
@@
     )
   )
-  (global_label "+3V3" (shape input) (at 102.87 134.62 180) (fields_autoplaced)
+  (global_label "+3V3" (shape input) (at 116.84 134.62 180) (fields_autoplaced)
     (effects (font (size 1.27 1.27)) (justify right))
-    (property "Intersheetrefs" "${INTERSHEET_REFS}" (at 94.8048 134.62 0)
+    (property "Intersheetrefs" "${INTERSHEET_REFS}" (at 108.7748 134.62 0)
       (effects (font (size 1.27 1.27)) (justify right) hide)
     )

Commit message: replaced nrf 3.3v w/ 3v, added 3v power plane
Connections:
- net +3V: now also C12.1, C14.1, C19.1, C6.1, C7.1, C8.1, J1.1 (Pin_1), R10.1, U3.A22 (VDD), U3.AD14 (VDD), U3.AD23 (VDD), U3.B1 (VDD), U3.W1 (VDD), U3.Y2 (VDDH)
- net +3V3: no longer C12.1, C14.1, C19.1, C6.1, C7.1, C8.1, J1.1 (Pin_1), R10.1, U3.A22 (VDD), U3.AD14 (VDD), U3.AD23 (VDD), U3.B1 (VDD), U3.W1 (VDD), U3.Y2 (VDDH)
- net AD2: no longer names the net of U3.AD2 (VBUS)
Changed lines of the file:
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@@
   (no_connect (at 176.53 137.16))
   (no_connect (at 187.96 157.48))
+  (no_connect (at 176.53 170.18))
   (no_connect (at 271.78 172.72))
   (no_connect (at 176.53 127))
@@
   (no_connect (at 176.53 104.14))
   (no_connect (at 176.53 124.46))
-  (no_connect (at 176.53 165.1))
   (no_connect (at 271.78 101.6))
   (no_connect (at 123.19 232.41))
@@
   (no_connect (at 176.53 139.7))
   (no_connect (at 176.53 162.56))
+  (no_connect (at 176.53 165.1))
   (no_connect (at 271.78 86.36))
   (no_connect (at 271.78 170.18))
-  (no_connect (at 176.53 170.18))
   (no_connect (at 176.53 129.54))
   (no_connect (at 48.26 55.88))
@@
     (stroke (width 0) (type default))
   )
-  (wire (pts (xy 120.65 134.62) (xy 116.84 134.62))
+  (wire (pts (xy 120.65 134.62) (xy 102.87 134.62))
     (stroke (width 0) (type default))
   )
@@
   (label "OSCB" (at 90.17 76.2 180) (fields_autoplaced)
     (effects (font (size 1.27 1.27)) (justify right bottom))
-  )
-  (label "AD2" (at 176.53 165.1 0) (fields_autoplaced)
-    (effects (font (size 1.27 1.27)) (justify left bottom))
   )
   (label "INT1" (at 48.26 58.42 0) (fields_autoplaced)
@@
     )
   )
-  (global_label "+3V3" (shape input) (at 289.56 95.25 90) (fields_autoplaced)
-    (effects (font (size 1.27 1.27)) (justify left))
-    (property "Intersheetrefs" "${INTERSHEET_REFS}" (at 289.56 87.1848 90)
+  (global_label "+3V" (shape input) (at 289.56 95.25 90) (fields_autoplaced)
+    (effects (font (size 1.27 1.27)) (justify left))
+    (property "Intersheetrefs" "${INTERSHEET_REFS}" (at 289.56 88.3943 90)
       (effects (font (size 1.27 1.27)) (justify left) hide)
     )
@@
     )
   )
-  (global_label "+3V3" (shape input) (at 116.84 134.62 180) (fields_autoplaced)
+  (global_label "+3V" (shape input) (at 102.87 134.62 180) (fields_autoplaced)
     (effects (font (size 1.27 1.27)) (justify right))
-    (property "Intersheetrefs" "${INTERSHEET_REFS}" (at 108.7748 134.62 0)
+    (property "Intersheetrefs" "${INTERSHEET_REFS}" (at 96.0143 134.62 0)
       (effects (font (size 1.27 1.27)) (justify right) hide)
     )
@@
     )
   )
-  (global_label "+3V3" (shape input) (at 107.95 149.86 90) (fields_autoplaced)
-    (effects (font (size 1.27 1.27)) (justify left))
-    (property "Intersheetrefs" "${INTERSHEET_REFS}" (at 107.95 141.7948 90)
-      (effects (font (size 1.27 1.27)) (justify left) hide)
-    )
-  )
-  (global_label "+3V3" (shape input) (at 85.09 132.08 180) (fields_autoplaced)
+  (global_label "+3V" (shape input) (at 107.95 149.86 90) (fields_autoplaced)
+    (effects (font (size 1.27 1.27)) (justify left))
+    (property "Intersheetrefs" "${INTERSHEET_REFS}" (at 107.95 143.0043 90)
+      (effects (font (size 1.27 1.27)) (justify left) hide)
+    )
+  )
+  (global_label "+3V" (shape input) (at 85.09 132.08 180) (fields_autoplaced)
     (effects (font (size 1.27 1.27)) (justify right))
-    (property "Intersheetrefs" "${INTERSHEET_REFS}" (at 77.0248 132.08 0)
+    (property "Intersheetrefs" "${INTERSHEET_REFS}" (at 78.2343 132.08 0)
       (effects (font (size 1.27 1.27)) (justify right) hide)
     )
@@
     )
   )
-  (global_label "+3V3" (shape input) (at 311.15 175.26 0) (fields_autoplaced)
-    (effects (font (size 1.27 1.27)) (justify left))
-    (property "Intersheetrefs" "${INTERSHEET_REFS}" (at 319.2152 175.26 0)
-      (effects (font (size 1.27 1.27)) (justify left) hide)
-    )
-  )
-  (global_label "+3V3" (shape input) (at 151.13 71.12 0) (fields_autoplaced)
-    (effects (font (size 1.27 1.27)) (justify left))
-    (property "Intersheetrefs" "${INTERSHEET_REFS}" (at 159.1952 71.12 0)
+  (global_label "+3V" (shape input) (at 311.15 175.26 0) (fields_autoplaced)
+    (effects (font (size 1.27 1.27)) (justify left))
+    (property "Intersheetrefs" "${INTERSHEET_REFS}" (at 318.0057 175.26 0)
+      (effects (font (size 1.27 1.27)) (justify left) hide)
+    )
+  )
+  (global_label "+3V" (shape input) (at 151.13 71.12 0) (fields_autoplaced)
+    (effects (font (size 1.27 1.27)) (justify left))
+    (property "Intersheetrefs" "${INTERSHEET_REFS}" (at 157.9857 71.12 0)
       (effects (font (size 1.27 1.27)) (justify left) hide)
     )
@@
     )
   )
-  (global_label "+3V3" (shape input) (at 278.13 76.2 180) (fields_autoplaced)
+  (global_label "+3V" (shape input) (at 278.13 76.2 180) (fields_autoplaced)
     (effects (font (size 1.27 1.27)) (justify right))
-    (property "Intersheetrefs" "${INTERSHEET_REFS}" (at 270.0648 76.2 0)
+    (property "Intersheetrefs" "${INTERSHEET_REFS}" (at 271.2743 76.2 0)
       (effects (font (size 1.27 1.27)) (justify right) hide)
     )
